File: Gem.kicad_pcb (KiCad board)
At the start: 2 copper layers, 76.2 x 54.6 mm, 39 parts, among them IC1 AD8226, IC2 AD8538ARZ, M1 ALLSENSORS-A6AAF-CUTLEADS, M2 DIAVOLINO, M3 POLOLU-MICROSD, M4 POLOLU-REGULATOR-MOD, M5 ADAFRUIT-ADS1115-MOD, M6 ADAFRUIT-GPS-MOD

Commit message: v0.83, last version using Diavolino
Other:
- board text added: "Gem 0.83"
- board text removed: "Gem 0.82"

Commit message: v0.9, first version using Efficientino
Parts:
- removed 2-11V37, GND37: WIREPAD2,15/1,0, 2_15_1_0
- removed C7: 0.1uF, C025-024X044
- removed M3: POLOLU-MICROSD, POLOLU-MICROSD
- removed M4: POLOLU-REGULATOR-MOD, POLOLU-ADJUSTABLE-REGULATOR-MOD
- removed M5: ADAFRUIT-ADS1115-MOD, ADAFRUIT-ADS1115-MOD
- removed hole: VAL**, hole
- added C10: 0.1uF, Capacitors_SMD:C_0805, B.Cu at (48.8, 23.0)
- added F6: FB, Capacitors_SMD:C_0805, F.Cu at (24.6, 48.6)
- added F7: FB, Capacitors_SMD:C_0805, B.Cu at (3.17, 9.78)
- added R11: 2.2k, Resistors_SMD:R_0805, F.Cu at (54.1, 45.6)
- added R12: 2.2k, Resistors_SMD:R_0805, F.Cu at (54.1, 47.6)
- added U1: ADS1115, Housings_SSOP:MSOP-10_3x3mm_Pitch0.5mm, F.Cu at (41.1, 36.7)
- added U2: TCR2EF, Gem-modular:SC-74A, F.Cu at (27.9, 47.4)
- added U3: Micro-SD, Gem-modular:Micro-SD, F.Cu at (0.89, 19.7)
- C1: footprint C025-024X044 -> Gem-modular:C025-024X044
- C2: value 100uF -> 0.1uF; footprint E3_5-8 -> Capacitors_SMD:C_0805
- C3, C4, C5, C6: footprint C025-024X044 -> Capacitors_SMD:C_0805; moved to F.Cu
- C8: footprint C025-024X044 -> Capacitors_SMD:C_0805
- C9: value 22uF -> 22 uF; footprint C050-024X044 -> Capacitors_SMD:C_0805; moved to F.Cu
- F1: footprint FB -> Capacitors_SMD:C_0805
- F2, F3, F4, F5: footprint FB -> Capacitors_SMD:C_0805; moved to F.Cu
- IC1: footprint SO8 -> Gem-modular:SO8
- IC2: value AD8538ARZ -> AD8538; footprint SO8 -> Gem-modular:SO8
- M1: footprint ALLSENSORS-A6AAF-CUTLEADS -> Gem-modular:ALLSENSORS-A6AAF-CUTLEADS
- M2: footprint ARDUINO-NOHOLE-DIM_ON_BDOCU_ONLY_movetext -> Gem-modular:ARDUINO-NOHOLE-DIM_ON_BDOCU_ONLY
- M6: footprint ADAFRUIT-ULTIMATE-GPS-MOD -> Gem-modular:ADAFRUIT-ULTIMATE-GPS-MOD
- R1, R2: footprint 0204_5 -> Resistors_SMD:R_0805
- R10, R4, R5, R6, R7, R8, R9: footprint 0204_5 -> Resistors_SMD:R_0805; moved to F.Cu
- R3: footprint 0204_7 -> Gem-modular:0204_5
- S1: footprint EG1218 -> Gem-modular:EG1218
- TMP36: footprint TO92-EBC-OVAL -> Gem-modular:TO92-EBC-OVAL
- red1: footprint LED3MM -> Gem-modular:LED3MM
- moved C2 51.1 mm to (21.0, 48.6)
- moved C5 31.7 mm to (42.7, 39.5), turned to 0 degrees
- moved F3 31.4 mm to (42.7, 41.3), turned to 0 degrees
- moved R10 18.3 mm to (22.9, 19.1)
- moved C9 18.3 mm to (24.6, 46.1)
- moved R4 18.3 mm to (26.4, 28.1), turned to 90 degrees
- moved R5 15.4 mm to (24.1, 28.1), turned to 270 degrees
- moved C8 14.1 mm to (5.59, 9.65), turned to 270 degrees
- moved IC2 13.7 mm to (31.8, 28.6)
- moved TMP36 12.5 mm to (37.6, 44.1), turned to 0 degrees
- moved S1 11.3 mm to (26.4, 15.9), turned to 0 degrees
- moved C4 9.02 mm to (30.7, 24.3), turned to 0 degrees
- moved F2 8.21 mm to (26.7, 24.3), turned to 0 degrees
- moved R7 8.21 mm to (42.7, 6.86)
- moved R6 8.18 mm to (42.7, 9.14), turned to 0 degrees
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Connections:
- C4 pad 1: /N$30 -> /N$29
- C5 pad 1: /N$29 -> GND
- C5 pad 2: GND -> Net-(C5-Pad2)
- C8 pad 1: +3V3 -> GND
- C8 pad 2: GND -> Net-(C8-Pad2)
- C9 pad 1: +3V3 -> VAA
- IC1 pad 6: /N$10 -> +1V5
- IC2 pad 2: /N$10 -> +1V5
- IC2 pad 6: /N$10 -> +1V5
- IC2 pad 7: /N$30 -> /N$29
- M1 pad 1: (no net) -> +1V5
- M2 pad 5V: +3V3 -> Net-(M2-Pad5V)
- M2 pad A2: (no net) -> Net-(M2-PadA2)
- M2 pad A3: (no net) -> Net-(M2-PadA3)
- M2 pad AREF: (no net) -> VAA
- M2 pad D3: (no net) -> Net-(M2-PadD3)
- M2 pad D7: (no net) -> Net-(M2-PadD7)
- M2 pad D8: (no net) -> Net-(M2-PadD8)
- M2 pad D9: (no net) -> Net-(M2-PadD9)
- M2 pad RESE: (no net) -> Net-(M2-PadRESE)
- M2 pad VIN: (no net) -> +BATT
- R8 pad 1: /N$1 -> +BATT
- TMP36 pad E: +3V3 -> VAA
Routing:
- net VAA: track 0.00 -> 63.9 mm, vias 0 -> 2
- net /N$10: track 57.6 -> 0.00 mm
- net /N$1: track 48.5 -> 0.00 mm
- net +1V5: track 0.00 -> 36.1 mm, vias 0 -> 1
- net /N$2: track 26.8 -> 4.86 mm
- net GND: track 3.24 -> 25.1 mm, vias 2 -> 15
- net /N$11: track 24.3 -> 41.4 mm, vias 0 -> 2
- net /N$27: track 22.1 -> 9.11 mm
- net /N$25: track 25.2 -> 14.0 mm
- net /N$5: track 12.1 -> 2.53 mm
- net +BATT: track 0.00 -> 6.88 mm
- net /N$30: track 6.31 -> 0.00 mm
- net Net-(C5-Pad2): track 0.00 -> 6.01 mm
- net /N$12: track 31.1 -> 25.2 mm
- net /N$18: track 23.5 -> 28.8 mm
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- added copper zone on F.Cu, net VAA
Other:
- board size 76.2 x 54.6 mm -> 60.2 x 54 mm
- net class Default: clearance 0.3048 -> 0.1524; trace_width 0.4064 -> 0.254
- rule trace_clearance: 0.3048 -> 0.1524
- rule trace_min: 0.4064 -> 0.1524
- board text added: "Gem 0.9"
- board text removed: "Buffered Reference"
- board text removed: "Gem 0.83"
- board text removed: "Instr Amp"
- board text removed: "RC Filter"

Commit message: v0.91
Parts:
- removed C10: 0.1uF, Capacitors_SMD:C_0805
- added C7: 0.1uF, Capacitors_SMD:C_0805, F.Cu at (5.33, 3.81)
- C1: value 15nF -> 0.1uF; footprint Gem-modular:C025-024X044 -> Capacitors_SMD:C_0805
- C8: value 0.1uF -> 22 uF; moved to F.Cu
- C9: value 22 uF -> 15nF; footprint Capacitors_SMD:C_0805 -> Gem-modular:C025-024X044
- F1, F7: moved to F.Cu
- R10: value 470 -> 100k
- R3: value 2.2k -> 47k; footprint Gem-modular:0204_5 -> Resistors_SMD:R_0805
- R5: value 47k -> 2.2k; footprint Resistors_SMD:R_0805 -> Gem-modular:R-TH-VERT
- R8: value 100k -> 470
- blue1: footprint LED3MM -> Gem-modular:LED3MM
- moved C8 44.6 mm to (33.3, 44.6), turned to 0 degrees
- moved R10 36.4 mm to (45.5, 47.6), turned to 0 degrees
- moved R8 34.6 mm to (24.6, 19.1)
- moved C6 32.5 mm to (49.0, 29.6), turned to 180 degrees
- moved F4 32.0 mm to (45.2, 41.4)
- moved F6 29.8 mm to (49.0, 31.5), turned to 180 degrees
- moved F1 29.6 mm to (19.2, 25.3), turned to 0 degrees
- moved C2 24.7 mm to (40.4, 33.4), turned to 0 degrees
- moved F3 21.2 mm to (29.1, 25.0)
- moved C4 21.0 mm to (45.2, 39.5)
- moved F5 18.1 mm to (29.3, 48.1)
- moved F2 15.5 mm to (40.4, 31.5)
- moved C5 14.9 mm to (29.3, 46.2)
- moved C1 14.6 mm to (19.2, 27.2), turned to 0 degrees
- moved C3 9.77 mm to (33.3, 25.0)
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Connections:
- C1 pad 1: /N$9 -> /N$32
- C1 pad 2: /N$4 -> GND
- C2 pad 1: +3V3 -> /N$31
- C3 pad 1: /N$31 -> /N$29
- C4 pad 1: /N$29 -> GND
- C4 pad 2: GND -> Net-(C4-Pad2)
- C6 pad 1: /N$32 -> GND
- C6 pad 2: GND -> /N$28
- C8 pad 1: GND -> VAA
- C8 pad 2: Net-(C8-Pad2) -> GND
- C9 pad 1: VAA -> /N$9
- C9 pad 2: GND -> /N$4
- F1 pad 1: +3V3 -> /N$32
- F1 pad 2: /N$28 -> VAA
- F2 pad 1: VAA -> /N$31
- F2 pad 2: /N$29 -> VAA
- F3 pad 2: Net-(C5-Pad2) -> /N$29
- F4 pad 1: /N$32 -> VAA
- F4 pad 2: VAA -> Net-(C4-Pad2)
- F5 pad 1: /N$31 -> +3V3
- F5 pad 2: VAA -> Net-(C5-Pad2)
- F6 pad 2: Net-(F6-Pad2) -> /N$28
- F7 pad 1: Net-(C8-Pad2) -> Net-(C7-Pad2)
- R10 pad 1: /N$26 -> +BATT
- R10 pad 2: +3V3 -> /N$27
- R3 pad 1: /N$5 -> GND
- R3 pad 2: /N$6 -> /N$8
- R5 pad 1: GND -> /N$5
- R5 pad 2: /N$8 -> /N$6
- R8 pad 1: +BATT -> /N$26
- R8 pad 2: /N$27 -> +3V3
- U1 pad 8: Net-(C5-Pad2) -> Net-(C4-Pad2)
- U2 pad 1: Net-(F6-Pad2) -> Net-(C5-Pad2)
- U3 pad 4: Net-(C8-Pad2) -> Net-(C7-Pad2)
Routing:
- net VAA: track 63.9 -> 23.4 mm, vias 2 -> 1
- net /N$11: track 41.4 -> 26.7 mm, vias 2 -> 0
- net Net-(C7-Pad2): track 0.00 -> 11.6 mm
- net GND: track 25.1 -> 36.7 mm, vias 15 -> 14
- net Net-(C4-Pad2): track 0.00 -> 6.01 mm
- net /N$32: track 15.0 -> 9.15 mm
- net /N$14: track 20.5 -> 16.5 mm
- net /N$13: track 24.9 -> 21.0 mm
- net Net-(C8-Pad2): track 3.86 -> 0.00 mm, vias 1 -> 0
- net /N$28: track 5.15 -> 8.46 mm
- net +1V5: track 36.1 -> 32.8 mm
- net +3V3: track 2.55 -> 4.93 mm, vias 2 -> 0
- net Net-(C5-Pad2): track 6.01 -> 3.78 mm
- net +BATT: track 6.88 -> 8.71 mm
- net /N$12: track 25.2 -> 23.6 mm
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Other:
- board size 60.2 x 54 mm -> 56 x 54 mm
- board text added: "For use with 3.3V systems only. Running at 5V will damage the SD card and possibly the GPS."
- board text added: "Gem 0.91"
- board text removed: "Gem 0.9"

Commit message: v0.92, version of SRL paper
Parts:
- M2: value DIAVOLINO -> Board
- M6: value ADAFRUIT-GPS-MOD -> ADAFRUIT-GPS
- moved R8 5.15 mm to (29.8, 19.3)
- moved TMP36 0.64 mm to (40.8, 44.1)
- moved C1 0.64 mm to (19.8, 27.2)
- moved F1 0.64 mm to (19.8, 25.3)
- moved F3 0.64 mm to (29.7, 25.0)
- moved R1 0.64 mm to (25.5, 36.2)
- moved R2 0.64 mm to (25.5, 39.8)
- moved R3 0.64 mm to (27.6, 28.8)
- moved R4 0.64 mm to (29.6, 28.8)
- moved R5 0.64 mm to (30.7, 34.0)
- moved M1 0.63 mm to (6.35, 36.7)
- moved C2 0.63 mm to (41.0, 33.4)
- moved C3 0.63 mm to (33.9, 25.0)
- moved C4 0.63 mm to (45.8, 39.5)
- moved C9 0.63 mm to (27.8, 38.4)
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Connections:
- M2 pad 5V: Net-(M2-Pad5V) -> (no net)
- M2 pad A2: Net-(M2-PadA2) -> (no net)
- M2 pad A3: Net-(M2-PadA3) -> (no net)
- M2 pad D3: Net-(M2-PadD3) -> (no net)
- M2 pad D7: Net-(M2-PadD7) -> (no net)
- M2 pad D8: Net-(M2-PadD8) -> (no net)
- M2 pad D9: Net-(M2-PadD9) -> (no net)
- M2 pad RESE: Net-(M2-PadRESE) -> (no net)
- U1 pad 1: Net-(U1-Pad1) -> (no net)
- U1 pad 2: Net-(U1-Pad2) -> (no net)
- U1 pad 6: Net-(U1-Pad6) -> (no net)
- U1 pad 7: Net-(U1-Pad7) -> (no net)
- U2 pad 4: Net-(U2-Pad4) -> (no net)
- U3 pad 1: Net-(U3-Pad1) -> (no net)
- U3 pad 8: Net-(U3-Pad8) -> (no net)
- U3 pad 9: Net-(U3-Pad9) -> (no net)
Routing:
- net VAA: track 23.4 -> 24.3 mm
- net +1V5: track 32.8 -> 33.6 mm
- net /N$15: track 20.3 -> 20.9 mm
- net /N$20: track 19.5 -> 18.9 mm
Other:
- board text added: "Gem 0.92"
- board text removed: "Gem 0.91"

Commit message: v0.92, libraries fixed
Parts:
- C9: footprint Gem-modular:C025-024X044 -> Gem:C025-024X044
- IC1, IC2: footprint Gem-modular:SO8 -> Gem:SO8
- M1: footprint Gem-modular:ALLSENSORS-A6AAF-CUTLEADS -> Gem:ALLSENSORS-A6AAF-CUTLEADS
- M2: footprint Gem-modular:ARDUINO-NOHOLE-DIM_ON_BDOCU_ONLY -> Gem:ARDUINO-NOHOLE-DIM_ON_BDOCU_ONLY
- M6: footprint Gem-modular:ADAFRUIT-ULTIMATE-GPS-MOD -> Gem:ADAFRUIT-ULTIMATE-GPS-MOD
- R5: footprint Gem-modular:R-TH-VERT -> Gem:R-TH-VERT
- S1: footprint Gem-modular:EG1218 -> Gem:EG1218
- TMP36: footprint Gem-modular:TO92-EBC-OVAL -> Gem:TO92-EBC-OVAL
- U2: footprint Gem-modular:SC-74A -> Gem:SC-74A
- U3: footprint Gem-modular:Micro-SD -> Gem:Micro-SD
- blue1, red1: footprint Gem-modular:LED3MM -> Gem:LED3MM
Changed lines of the file:
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@@
     (add_net VAA)
   )
-  (module Gem-modular:ALLSENSORS-A6AAF-CUTLEADS (layer Top)
+  (module Gem:ALLSENSORS-A6AAF-CUTLEADS (layer Top)
     (at 6.35 36.703 270)
     (attr virtual)
@@
     (pad "" np_thru_hole circle (at 10.795 0 270) (size 3.4 3.4) (drill 3.4) (layers *.Cu *.Mask))
   )
-  (module Gem-modular:ARDUINO-NOHOLE-DIM_ON_BDOCU_ONLY locked (layer Top)
+  (module Gem:ARDUINO-NOHOLE-DIM_ON_BDOCU_ONLY locked (layer Top)
     (at 57.15 1.7145)
     (attr virtual)
@@
       (net 33 +BATT))
   )
-  (module Gem-modular:EG1218 (layer Top)
+  (module Gem:EG1218 (layer Top)
     (at 26.289 15.875 180)
     (fp_text reference S1 (at 5.7785 -3.556 360) (layer F.SilkS)
@@
       (net 31 GND))
   )
-  (module Gem-modular:ADAFRUIT-ULTIMATE-GPS-MOD (layer Top)
+  (module Gem:ADAFRUIT-ULTIMATE-GPS-MOD (layer Top)
     (at 58.3565 21.717)
     (attr virtual)
@@
       (net 20 /N$28))
   )
-  (module Gem-modular:SO8 (layer Top)
+  (module Gem:SO8 (layer Top)
     (at 35.687 37.211 270)
     (descr "8-LEAD SMALL OUTLINE IC (SO-8)")
@@
       (net 23 /N$31))
   )
-  (module Gem-modular:SO8 (layer Top)
+  (module Gem:SO8 (layer Top)
     (at 34.925 29.337 270)
     (descr "8-LEAD SMALL OUTLINE IC (SO-8)")
@@
     )
   )
-  (module Gem-modular:SC-74A (layer Top)
+  (module Gem:SC-74A (layer Top)
     (at 33.147 47.371)
     (fp_text reference U2 (at 2.286 -0.127 90) (layer F.SilkS)
@@
       (net 34 "Net-(C5-Pad2)"))
   )
-  (module Gem-modular:LED3MM (layer Top)
+  (module Gem:LED3MM (layer Top)
     (at 37.338 18.796 270)
     (descr LED)
@@
       (net 31 GND))
   )
-  (module Gem-modular:LED3MM (layer Top)
+  (module Gem:LED3MM (layer Top)
     (at 37.338 12.954 270)
     (descr LED)
@@
       (net 31 GND))
   )
-  (module Gem-modular:Micro-SD (layer Top)
+  (module Gem:Micro-SD (layer Top)
     (at 2.921 19.685 90)
     (fp_text reference U3 (at 3.048 7.366 180) (layer F.SilkS)
@@
       (net 31 GND))
   )
-  (module Gem-modular:TO92-EBC-OVAL (layer Top)
+  (module Gem:TO92-EBC-OVAL (layer Top)
     (at 40.767 44.069)
     (descr TO-92)
@@
     )
   )
-  (module Gem-modular:C025-024X044 (layer Top)
+  (module Gem:C025-024X044 (layer Top)
     (at 27.813 38.354 90)
     (descr CAPACITOR)
@@
     )
   )
-  (module Gem-modular:R-TH-VERT (layer Top)
+  (module Gem:R-TH-VERT (layer Top)
     (at 30.734 34.036 90)
     (fp_text reference R5 (at -5.588 -0.127 180) (layer F.SilkS)
